Commit message: fix some porblems

File: src/robotiq_description/urdf/test.urdf (robot description, URDF)
Before this commit: robot robotiq_gripper, 10 links, 9 joints
Links:
- link robotiq_85_base_link: geometry collision mesh filename=file:///home/xiaobaige/ros2_moveit2_ur5e_grasp/install/robo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; visual mesh filename=file:///home/xiaobaige/ros2_moveit2_ur5e_grasp/install/robo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
- link robotiq_85_left_finger_link: geometry collision mesh filename=file:///home/xiaobaige/ros2_moveit2_ur5e_grasp/install/robo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; visual mesh filename=file:///home/xiaobaige/ros2_moveit2_ur5e_grasp/install/robo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
- link robotiq_85_left_finger_tip_link: geometry collision mesh filename=file:///home/xiaobaige/ros2_moveit2_ur5e_grasp/install/robo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; visual mesh filename=file:///home/xiaobaige/ros2_moveit2_ur5e_grasp/install/robo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
- link robotiq_85_left_inner_knuckle_link: geometry collision mesh filename=file:///home/xiaobaige/ros2_moveit2_ur5e_grasp/install/robo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; visual mesh filename=file:///home/xiaobaige/ros2_moveit2_ur5e_grasp/install/robo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
- link robotiq_85_left_knuckle_link: geometry collision mesh filename=file:///home/xiaobaige/ros2_moveit2_ur5e_grasp/install/robo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; visual mesh filename=file:///home/xiaobaige/ros2_moveit2_ur5e_grasp/install/robo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
- link robotiq_85_right_finger_link: geometry collision mesh filename=file:///home/xiaobaige/ros2_moveit2_ur5e_grasp/install/robo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; visual mesh filename=file:///home/xiaobaige/ros2_moveit2_ur5e_grasp/install/robo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
- link robotiq_85_right_finger_tip_link: geometry collision mesh filename=file:///home/xiaobaige/ros2_moveit2_ur5e_grasp/install/robo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; visual mesh filename=file:///home/xiaobaige/ros2_moveit2_ur5e_grasp/install/robo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
- link robotiq_85_right_inner_knuckle_link: geometry collision mesh filename=file:///home/xiaobaige/ros2_moveit2_ur5e_grasp/install/robo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; visual mesh filename=file:///home/xiaobaige/ros2_moveit2_ur5e_grasp/install/robo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
- link robotiq_85_right_knuckle_link: geometry collision mesh filename=file:///home/xiaobaige/ros2_moveit2_ur5e_grasp/install/robo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; visual mesh filename=file:///home/xiaobaige/ros2_moveit2_ur5e_grasp/install/robo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

File: src/ur5e_gripper_description/urdf/ur5e_gripper.urdf (robot description, URDF)
Before this commit: robot ur5e_gripper, 27 links, 26 joints
Links:
- link base_link_inertia: geometry collision mesh filename=file:///home/xiaobaige/ros2_moveit2_ur5e_grasp/install/ur_d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; visual mesh filename=file:///home/xiaobaige/ros2_moveit2_ur5e_grasp/install/ur_d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
- link forearm_link: geometry collision mesh filename=file:///home/xiaobaige/ros2_moveit2_ur5e_grasp/install/ur_d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; visual mesh filename=file:///home/xiaobaige/ros2_moveit2_ur5e_grasp/install/ur_d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
- link robotiq_85_base_link: geometry collision mesh filename=file:///home/xiaobaige/ros2_moveit2_ur5e_grasp/install/robo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; visual mesh filename=file:///home/xiaobaige/ros2_moveit2_ur5e_grasp/install/robo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
- link robotiq_85_left_finger_link: geometry collision mesh filename=file:///home/xiaobaige/ros2_moveit2_ur5e_grasp/install/robo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; visual mesh filename=file:///home/xiaobaige/ros2_moveit2_ur5e_grasp/install/robo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
- link robotiq_85_left_finger_tip_link: geometry collision mesh filename=file:///home/xiaobaige/ros2_moveit2_ur5e_grasp/install/robo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; visual mesh filename=file:///home/xiaobaige/ros2_moveit2_ur5e_grasp/install/robo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
- link robotiq_85_left_inner_knuckle_link: geometry collision mesh filename=file:///home/xiaobaige/ros2_moveit2_ur5e_grasp/install/robo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; visual mesh filename=file:///home/xiaobaige/ros2_moveit2_ur5e_grasp/install/robo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
- link robotiq_85_left_knuckle_link: geometry collision mesh filename=file:///home/xiaobaige/ros2_moveit2_ur5e_grasp/install/robo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; visual mesh filename=file:///home/xiaobaige/ros2_moveit2_ur5e_grasp/install/robo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
- link robotiq_85_right_finger_link: geometry collision mesh filename=file:///home/xiaobaige/ros2_moveit2_ur5e_grasp/install/robo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; visual mesh filename=file:///home/xiaobaige/ros2_moveit2_ur5e_grasp/install/robo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
- link robotiq_85_right_finger_tip_link: geometry collision mesh filename=file:///home/xiaobaige/ros2_moveit2_ur5e_grasp/install/robo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; visual mesh filename=file:///home/xiaobaige/ros2_moveit2_ur5e_grasp/install/robo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
- link robotiq_85_right_inner_knuckle_link: geometry collision mesh filename=file:///home/xiaobaige/ros2_moveit2_ur5e_grasp/install/robo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; visual mesh filename=file:///home/xiaobaige/ros2_moveit2_ur5e_grasp/install/robo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
- link robotiq_85_right_knuckle_link: geometry collision mesh filename=file:///home/xiaobaige/ros2_moveit2_ur5e_grasp/install/robo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; visual mesh filename=file:///home/xiaobaige/ros2_moveit2_ur5e_grasp/install/robo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
- link shoulder_link: geometry collision mesh filename=file:///home/xiaobaige/ros2_moveit2_ur5e_grasp/install/ur_d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; visual mesh filename=file:///home/xiaobaige/ros2_moveit2_ur5e_grasp/install/ur_d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
- link upper_arm_link: geometry collision mesh filename=file:///home/xiaobaige/ros2_moveit2_ur5e_grasp/install/ur_d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; visual mesh filename=file:///home/xiaobaige/ros2_moveit2_ur5e_grasp/install/ur_d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
- link wrist_1_link: geometry collision mesh filename=file:///home/xiaobaige/ros2_moveit2_ur5e_grasp/install/ur_d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; visual mesh filename=file:///home/xiaobaige/ros2_moveit2_ur5e_grasp/install/ur_d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
- link wrist_2_link: geometry collision mesh filename=file:///home/xiaobaige/ros2_moveit2_ur5e_grasp/install/ur_d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; visual mesh filename=file:///home/xiaobaige/ros2_moveit2_ur5e_grasp/install/ur_d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
- link wrist_3_link: geometry collision mesh filename=file:///home/xiaobaige/ros2_moveit2_ur5e_grasp/install/ur_d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; visual mesh filename=file:///home/xiaobaige/ros2_moveit2_ur5e_grasp/install/ur_d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

Commit message: fix gazebo problems

File: src/robotiq_description/urdf/test.urdf (robot description, URDF)
Before this commit: robot robotiq_gripper, 10 links, 9 joints
Links:
- link robotiq_85_base_link: geometry collision mesh filename=file:///home/nack/UR5e_Vision_Assemble/install/robotiq_desc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; visual mesh filename=file:///home/nack/UR5e_Vision_Assemble/install/robotiq_desc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
- link robotiq_85_left_finger_link: geometry collision mesh filename=file:///home/nack/UR5e_Vision_Assemble/install/robotiq_desc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; visual mesh filename=file:///home/nack/UR5e_Vision_Assemble/install/robotiq_desc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
- link robotiq_85_left_finger_tip_link: geometry collision mesh filename=file:///home/nack/UR5e_Vision_Assemble/install/robotiq_desc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; visual mesh filename=file:///home/nack/UR5e_Vision_Assemble/install/robotiq_desc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
- link robotiq_85_left_inner_knuckle_link: geometry collision mesh filename=file:///home/nack/UR5e_Vision_Assemble/install/robotiq_desc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; visual mesh filename=file:///home/nack/UR5e_Vision_Assemble/install/robotiq_desc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
- link robotiq_85_left_knuckle_link: geometry collision mesh filename=file:///home/nack/UR5e_Vision_Assemble/install/robotiq_desc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; visual mesh filename=file:///home/nack/UR5e_Vision_Assemble/install/robotiq_desc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
- link robotiq_85_right_finger_link: geometry collision mesh filename=file:///home/nack/UR5e_Vision_Assemble/install/robotiq_desc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; visual mesh filename=file:///home/nack/UR5e_Vision_Assemble/install/robotiq_desc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
- link robotiq_85_right_finger_tip_link: geometry collision mesh filename=file:///home/nack/UR5e_Vision_Assemble/install/robotiq_desc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; visual mesh filename=file:///home/nack/UR5e_Vision_Assemble/install/robotiq_desc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
- link robotiq_85_right_inner_knuckle_link: geometry collision mesh filename=file:///home/nack/UR5e_Vision_Assemble/install/robotiq_desc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; visual mesh filename=file:///home/nack/UR5e_Vision_Assemble/install/robotiq_desc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
- link robotiq_85_right_knuckle_link: geometry collision mesh filename=file:///home/nack/UR5e_Vision_Assemble/install/robotiq_desc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; visual mesh filename=file:///home/nack/UR5e_Vision_Assemble/install/robotiq_desc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

File: src/ur5e_gripper_description/urdf/ur5e_gripper.urdf (robot description, URDF)
Before this commit: robot ur5e_gripper, 27 links, 26 joints
Links:
- link base_link_inertia: geometry collision mesh filename=file:///home/nack/UR5e_Vision_Assemble/install/ur_descripti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; visual mesh filename=file:///home/nack/UR5e_Vision_Assemble/install/ur_descripti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
- link forearm_link: geometry collision mesh filename=file:///home/nack/UR5e_Vision_Assemble/install/ur_descripti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; visual mesh filename=file:///home/nack/UR5e_Vision_Assemble/install/ur_descripti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
- link robotiq_85_base_link: geometry collision mesh filename=file:///home/nack/UR5e_Vision_Assemble/install/robotiq_desc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; visual mesh filename=file:///home/nack/UR5e_Vision_Assemble/install/robotiq_desc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
- link robotiq_85_left_finger_link: geometry collision mesh filename=file:///home/nack/UR5e_Vision_Assemble/install/robotiq_desc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; visual mesh filename=file:///home/nack/UR5e_Vision_Assemble/install/robotiq_desc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
- link robotiq_85_left_finger_tip_link: geometry collision mesh filename=file:///home/nack/UR5e_Vision_Assemble/install/robotiq_desc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; visual mesh filename=file:///home/nack/UR5e_Vision_Assemble/install/robotiq_desc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
- link robotiq_85_left_inner_knuckle_link: geometry collision mesh filename=file:///home/nack/UR5e_Vision_Assemble/install/robotiq_desc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; visual mesh filename=file:///home/nack/UR5e_Vision_Assemble/install/robotiq_desc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
- link robotiq_85_left_knuckle_link: geometry collision mesh filename=file:///home/nack/UR5e_Vision_Assemble/install/robotiq_desc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; visual mesh filename=file:///home/nack/UR5e_Vision_Assemble/install/robotiq_desc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
- link robotiq_85_right_finger_link: geometry collision mesh filename=file:///home/nack/UR5e_Vision_Assemble/install/robotiq_desc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; visual mesh filename=file:///home/nack/UR5e_Vision_Assemble/install/robotiq_desc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
- link robotiq_85_right_finger_tip_link: geometry collision mesh filename=file:///home/nack/UR5e_Vision_Assemble/install/robotiq_desc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; visual mesh filename=file:///home/nack/UR5e_Vision_Assemble/install/robotiq_desc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
- link robotiq_85_right_inner_knuckle_link: geometry collision mesh filename=file:///home/nack/UR5e_Vision_Assemble/install/robotiq_desc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; visual mesh filename=file:///home/nack/UR5e_Vision_Assemble/install/robotiq_desc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
- link robotiq_85_right_knuckle_link: geometry collision mesh filename=file:///home/nack/UR5e_Vision_Assemble/install/robotiq_desc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; visual mesh filename=file:///home/nack/UR5e_Vision_Assemble/install/robotiq_desc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
- link shoulder_link: geometry collision mesh filename=file:///home/nack/UR5e_Vision_Assemble/install/ur_descripti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; visual mesh filename=file:///home/nack/UR5e_Vision_Assemble/install/ur_descripti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
- link upper_arm_link: geometry collision mesh filename=file:///home/nack/UR5e_Vision_Assemble/install/ur_descripti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; visual mesh filename=file:///home/nack/UR5e_Vision_Assemble/install/ur_descripti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
- link wrist_1_link: geometry collision mesh filename=file:///home/nack/UR5e_Vision_Assemble/install/ur_descripti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; visual mesh filename=file:///home/nack/UR5e_Vision_Assemble/install/ur_descripti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
- link wrist_2_link: geometry collision mesh filename=file:///home/nack/UR5e_Vision_Assemble/install/ur_descripti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; visual mesh filename=file:///home/nack/UR5e_Vision_Assemble/install/ur_descripti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
- link wrist_3_link: geometry collision mesh filename=file:///home/nack/UR5e_Vision_Assemble/install/ur_descripti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; visual mesh filename=file:///home/nack/UR5e_Vision_Assemble/install/ur_descripti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
